File: InitialConcepts/nanovoltmeter_fe.kicad_sch (KiCad schematic)
At the start: 125 parts, among them J1 INPUT_Cu_posts, J2 PWR +/-12V, J3 CTRL (isolated), K3 TQ2-L2-5V SHORT, K4 TQ2-L2-5V CAL, K5 TQ2-L2-5V MODE, Q1 LSK389B-1/2, Q10 KSC1845FTA, Q11 MMBT5401, Q12 MMBT5401, Q13 BCP56-16, Q14 BCP56-16, Q15 MMBT5401, Q16 2N4117A clamp, Q17 2N4117A clamp, Q18 2N4117A clamp, Q19 2N4117A clamp, Q2 LSK389B-1/2, Q3 LSK389B-1/2, Q4 LSK389B-1/2, Q5 LSK389B-1/2, Q6 LSK389B-1/2, Q7 LSK389B-1/2, Q8 LSK389B-1/2, Q9 KSC1845FTA, U1 OPA828IDR, U10 AQY221N2MY, U11 AQY221N2MY, U12 CPC1017N, U13 CPC1017N, U14 74LVC1G04, U15 74LVC1G04, U16 74LVC1G04, U17 74LVC1G04, U18 LTC2500-32, U19 LTC6655B-5, U2 OPA2210ID, U20 LP5907-2.5, U3 AD5689RBRUZ, U4 AQY221N2MY, U5 AQY221N2MY, U6 AQY221N2MY, U7 AQY221N2MY, U8 AQY221N2MY, U9 AQY221N2MY

Commit message: Working on front end protection and update teensy
Parts:
- removed K5: TQ2-L2-5V MODE, NVM:Relay_TQ2_THT, symbol Relay:AZ850P2-x
- added C32, C33: 100n, Capacitor_SMD:C_0805_2012Metric, symbol Device:C
- added Q20, Q21: DN2540N8 depl (norm-ON), NVM:SOT-89-3, symbol Device:Q_NJFET_DGS
- added Q22, Q23: 2N4117A clamp, NVM:TO-72-4, symbol Device:Q_NJFET_DGS
- added R49: 4k7, Resistor_SMD:R_0805_2012Metric, symbol Device:R
- added R50: 680R, Resistor_SMD:R_0805_2012Metric, symbol Device:R
- added R51: 52k3, Resistor_SMD:R_0805_2012Metric, symbol Device:R
- added R52, R54, R55: 10k, Resistor_SMD:R_0805_2012Metric, symbol Device:R
- added R53: 287k, Resistor_SMD:R_0805_2012Metric, symbol Device:R
- added R56: 100k, Resistor_SMD:R_0805_2012Metric, symbol Device:R
- added R57, R58: 390R, Resistor_SMD:R_0805_2012Metric, symbol Device:R
- added U21, U24, U25, U26, U27: AQY221N2MY, OptoDevice:Panasonic_APV-AQY_SSOP-4_4.45x2.65mm_P1.27mm, symbol Relay_SolidState:AQY282GS
- added U22: LM2903 (see note SEC7), Package_SO:SOIC-8_3.9x4.9mm_P1.27mm, symbol Comparator:LM2903
- added U23: 74LVC1G74 (trip latch), Package_TO_SOT_SMD:SOT-353_SC-70-5, symbol 74xGxx:74AUC1G74
- added U28: 74LVC1G04, Package_TO_SOT_SMD:SOT-23-5, symbol 74xGxx:74LVC1G04
Connections:
- net BR_LO is gone; now on net LO_F: U10.3, U11.3, U6.3, U7.3
- net +2V5: now also R51.1
- net +5VD: now also C32.1, C33.1, R50.1, R55.1, R57.1, R58.1, U22.8 (V+), U23.2 (D), U23.8 (VCC), U28.5 (VCC)
- net -12V_F: now also R49.2, R53.2
- net CH_A: now also U24.4, U25.4
- net HI_F: now also Q20.1 (D)
- net LO_F: now also U26.3, U27.3
- net RESET_N: now also U23.6 (~{CLR})
- net STAR: now also C32.2, C33.2, Q22.1 (D), Q22.3 (S), Q23.2 (G), R52.2, R54.1, U22.4 (V-), U23.1 (C), U23.4 (GND), U26.4, U27.4, U28.3 (GND)
- net BR_HI renamed HI_P
- net HI_P: now also Q21.1 (D), Q22.2 (G), Q23.1 (D), Q23.3 (S), U22.2 (-), U22.5 (+), U24.3, U25.3
- net K5_RST renamed FAULT_N
- net FAULT_N: now also U21.2, U23.3 (~{Q})
- net K5_SET renamed DIRECT_L
- net DIRECT_L: now also U28.2
- new net DIR_12: U24.2, U25.1
- new net DIR_34: U26.2, U27.1
- new net DIR_A1: R57.2, U24.1
- new net DIR_A2: R58.2, U26.1
- new net DIR_SINK: U25.2, U27.2, U28.4
- new net GPROT: Q20.2 (G), Q21.2 (G), R56.1, U21.4
- new net MIDP: Q20.3 (S), Q21.3 (S), R56.2
- new net N_TRIPA: R50.2, U21.1
- new net N_TRIPO: R49.1, U21.3
- new net TH_N: R53.1, R54.2, U22.6 (-)
- new net TH_P: R51.2, R52.1, U22.3 (+)
- new net TRIP_RAW: R55.2, U22.1, U22.7, U23.7 (~{PRE})
- no-connect marks 20 -> 21
Other:
- note added: "SEC 7 INPUT PROTECTION + FAIL-OPEN MODE (active). Q20/Q21 DN2540 depletion pair (norm-ON, ~3R each) in HI leg; Rg holds Vgs=0. HI_P clamp Q22/Q23 (2N4117A) to STAR. On |HI_P|>~0.4V window comp U22 sets latch U23 -> trip SSR U21 pulls GPROT to -12V => FETs OFF (true disconnect). K5 DELETED: mode via SSR pairs U24/U25 (direct HI_P->CH_A) + U26/U27 (LO_F->STAR); DIRECT_L high = direct mode; bridge U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"
