File: NVM_Digital_v1/NVM_Digital_v1.kicad_sch (KiCad schematic)
At the start: 30 parts, among them J7 DIN41612_M_3x8+8_Power_Male, Q1 DMG3415U, Q2 DMG3415U, Q3 DMG3415U, Q4 DMG3415U, U2 ISO7760F SPI/CTRL, U3 ISO7760F COILS 1-6, U4 ISO7762F COILS+RD, U44 CR2013-MI2120, U5 TBD62083AFWG

Commit message: Working on front end protection and update teensy
Parts:
- U4: value ISO7762F COILS+RD -> ISO7763F CTRL+RD
Connections:
- net STAR is gone; now on net LDAC_N: C2.2, C4.2, C6.2, C8.2, J7.P2, J7.P5, U2.9 (GND2), U3.9 (GND2), U4.9 (GND2), U5.9 (GND)
- net +5V_An: now also J7.c16
- net DGND: now also U4.3 (INB); no longer U4.5 (IND)
- net K5R_L: no longer U5.8 (I8)
- net LDAC_N: now reaches J7.c13
- net LDAC_N: now also U5.7 (I7), U5.8 (I8)
- net DIRECT_L: now reaches J7.c14
- net DIRECT_L: now also U4.15 (OUTA)
- net FAULT_N: now reaches J7.c15
- net FAULT_N: now also U4.12 (OUTD)
- net D_K5R renamed D_FAULT
- net D_FAULT: now also U4.5 (IND); no longer U4.3 (INB)
- net D_K5S renamed D_DIRECT
- removed net K5S_L: U4.15 (OUTA), U5.7 (I7)
- net K5_RST: no longer names the net of U5.11 (O8)
- net K5_RST: no longer J7.b16
- net K5_SET: no longer names the net of U5.12 (O7)
- net K5_SET: no longer J7.b15
- no-connect marks 25 -> 20
Other:
- note added: "(3) Floating-domain logic is 5V; Teensy side 3.3V via isolators. (4) Analog +/-12V goes to the FE only, via the DIN41612 (J7 P1/P4); STAR commons join at the FE board."
- note added: "SEC7 signals from FE J7 - IMPLEMENTED (U4 ISO7763F, Teensy 40/41): DIRECT_L (J7 c14): Teensy->FE mode-select level, HIGH=direct/high-Z, LOW=chop bridge. Route Teensy pin 40 -> isolator (DGND->floating) -> J7 c14. FAULT_N (J7 c15): FE->Teensy trip status, push-pull active-LOW (74LVC1G74 ~Q, not open-drain); U4 ISO7763F reverse ch-D -> Teensy pin 41 (INPUT_PULLUP). LDAC_N (J7 c13): tie LOW on FE, n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"
- note removed: "(3) Floating-domain logic is 5V; Teensy side 3.3V via isolators. (4) Analog +/-12V goes to FE J2 only; STAR commons join at the FE board."
Changed lines of the file:
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@@
 		)
 	)
-	(text "(3) Floating-domain logic is 5V; Teensy side 3.3V via isolators. (4) Analog +/-12V goes to FE J2 only; STAR commons join at the FE board."
+	(text "(3) Floating-domain logic is 5V; Teensy side 3.3V via isolators. (4) Analog +/-12V goes to the FE only, via the DIN41612 (J7 P1/P4); STAR commons join at the FE board."
 		(exclude_from_sim no)
 		(at 36.576 7.62 0)
@@
 		)
 	)
+	(text "SEC7 signals from FE J7 - IMPLEMENTED (U4 ISO7763F, Teensy 40/41):  DIRECT_L (J7 c14): Teensy->FE mode-select level, HIGH=direct/high-Z, LOW=chop bridge. Route Teensy pin 40 -> isolator (DGND->floating) -> J7 c14.  FAULT_N (J7 c15): FE->Teensy trip status, push-pull active-LOW (74LVC1G74 ~Q, not open-drain); U4 ISO7763F reverse ch-D -> Teensy pin 41 (INPUT_PULLUP).  LDAC_N (J7 c13): tie LOW on FE, no digital-side net.  COIL_COM (J7 c16): SSR/coil supply return, wire to +5V_An.  Also TBD: RESET_N line to clear the SEC7 trip latch (no Teensy pin assigned yet). Firmware ready: config.h PIN_DIRECT=40, PIN_FAULT=41."
+		(exclude_from_sim no)
+		(at 25.4 0 0)
+		(effects
+			(font
+				(size 1.6 1.6)
+				(color 200 0 0 1)
+			)
+			(justify left)
+		)
+	)
 	(junction
 		(at 96.52 119.38)
@@
 	)
 	(no_connect
-		(at 250.19 137.16)
-	)
-	(no_connect
 		(at 36.83 85.09)
 	)
@@
 	)
 	(no_connect
-		(at 250.19 129.54)
-	)
-	(no_connect
 		(at 62.23 85.09)
 	)
@@
 		(at 36.83 74.93)
 	)
-	(no_connect
-		(at 205.74 54.61)
-	)
-	(no_connect
-		(at 250.19 132.08)
-	)
-	(no_connect
-		(at 250.19 134.62)
-	)
 	(wire
 		(pts
@@
 	(wire
 		(pts
-			(xy 250.19 114.3) (xy 255.27 114.3)
-		)
-		(stroke
-			(width 0)
-			(type default)
-		)
-	)
-	(wire
-		(pts
 			(xy 30.48 46.99) (xy 36.83 46.99)
 		)
@@
 	(wire
 		(pts
-			(xy 250.19 116.84) (xy 255.27 116.84)
-		)
-		(stroke
-			(width 0)
-			(type default)
-		)
-	)
-	(wire
-		(pts
 			(xy 232.41 160.02) (xy 232.41 165.1)
 		)
@@
 		)
 	)
-	(global_label "K5_SET"
-		(shape passive)
-		(at 252.73 59.69 0)
-		(effects
-			(font
-				(size 1 1)
-			)
-			(justify left)
-		)
-		(property "Intersheetrefs" "${INTERSHEET_REFS}"
-			(at 252.73 59.69 0)
-			(hide yes)
-			(show_name no)
-			(do_not_autoplace no)
-			(effects
-				(font
-					(size 1.27 1.27)
-				)
-			)
-		)
-	)
-	(global_label "K5_SET"
-		(shape passive)
-		(at 255.27 114.3 0)
-		(effects
-			(font
-				(size 1 1)
-			)
-			(justify left)
-		)
-		(property "Intersheetrefs" "${INTERSHEET_REFS}"
-			(at 255.27 114.3 0)
-			(hide yes)
-			(show_name no)
-			(do_not_autoplace no)
-			(effects
-				(font
-					(size 1.27 1.27)
-				)
-			)
-		)
-	)
 	(global_label "TFT_CS"
 		(shape passive)
@@
 		)
 	)
-	(global_label "D_K5S"
+	(global_label "D_DIRECT"
 		(shape passive)
 		(at 30.48 64.77 180)
@@
 		)
 	)
-	(global_label "DGND"
+	(global_label "D_FAULT"
 		(shape passive)
 		(at 185.42 54.61 180)
@@
 		)
 	)
-	(global_label "D_K5R"
+	(global_label "DGND"
 		(shape passive)
 		(at 185.42 49.53 180)
@@
 		)
 	)
-	(global_label "D_K5S"
+	(global_label "D_DIRECT"
 		(shape passive)
 		(at 185.42 46.99 180)
@@
 		)
 	)
-	(global_label "K5R_L"
+	(global_label "STAR"
 		(shape passive)
 		(at 232.41 62.23 180)
@@
 		)
 	)
-	(global_label "K5S_L"
+	(global_label "STAR"
 		(shape passive)
 		(at 232.41 59.69 180)
@@
 		)
 	)
-	(global_label "K5S_L"
+	(global_label "DIRECT_L"
 		(shape passive)
 		(at 205.74 46.99 0)
@@
 		)
 	)
-	(global_label "K5_RST"
-		(shape passive)
-		(at 252.73 62.23 0)
-		(effects
-			(font
-				(size 1 1)
-			)
-			(justify left)
-		)
-		(property "Intersheetrefs" "${INTERSHEET_REFS}"
-			(at 252.73 62.23 0)
-			(hide yes)
-			(show_name no)
-			(do_not_autoplace no)
-			(effects
-				(font
-					(size 1.27 1.27)
-				)
-			)
-		)
-	)
 	(global_label "+5V_An"
 		(shape passive)
@@
 		)
 	)
-	(global_label "D_K5R"
+	(global_label "D_FAULT"
 		(shape passive)
 		(at 30.48 67.31 180)
@@
 		)
 	)
-	(global_label "K5_RST"
-		(shape passive)
-		(at 255.27 116.84 0)
-		(effects
-			(font
-				(size 1 1)
-			)
-			(justify left)
-		)
-		(property "Intersheetrefs" "${INTERSHEET_REFS}"
-			(at 255.27 116.84 0)
-			(hide yes)
-			(show_name no)
-			(do_not_autoplace no)
-			(effects
-				(font
-					(size 1.27 1.27)
-				)
-			)
-		)
-	)
 	(global_label "D_BL2"
 		(shape input)
@@
 			)
 		)
-		(property "Value" "ISO7762F COILS+RD"
+		(property "Value" "ISO7763F CTRL+RD"
 			(at 198.58 49.11 0)
 			(show_name no)
@@
 			)
 		)
-		(property "Description" "K5 coils forward; ADC SDOA + BUSY reverse"
+		(property "Description" "ISO7763F 3F/3R: DIRECT_L fwd (chA); reverse = ADC SDOA + BUSY + FAULT_N (chD). SWAP SYMBOL to 7763F variant."
 			(at 195.58 54.61 0)
 			(hide yes)
@@
 	)
 	(embedded_fonts no)
+	(wire
+		(pts
+			(xy 250.19 132.08) (xy 255.27 132.08)
+		)
+		(stroke
+			(width 0)
+			(type default)
+		)
+	)
+	(global_label "DIRECT_L"
+		(shape passive)
+		(at 255.27 132.08 0)
+		(effects
+			(font
+				(size 1 1)
+			)
+			(justify left)
+		)
+		(property "Intersheetrefs" "${INTERSHEET_REFS}"
+			(at 255.27 132.08 0)
+			(hide yes)
+			(show_name no)
+			(do_not_autoplace no)
+			(effects
+				(font
+					(size 1.27 1.27)
+				)
+			)
+		)
+	)
+	(wire
+		(pts
+			(xy 250.19 134.62) (xy 255.27 134.62)
+		)
+		(stroke
+			(width 0)
+			(type default)
+		)
+	)
+	(global_label "FAULT_N"
+		(shape passive)
+		(at 255.27 134.62 0)
+		(effects
+			(font
+				(size 1 1)
+			)
+			(justify left)
+		)
+		(property "Intersheetrefs" "${INTERSHEET_REFS}"
+			(at 255.27 134.62 0)
+			(hide yes)
+			(show_name no)
+			(do_not_autoplace no)
+			(effects
+				(font
+					(size 1.27 1.27)
+				)
+			)
+		)
+	)
+	(global_label "FAULT_N"
+		(shape passive)
+		(at 205.74 54.61 0)
+		(effects
+			(font
+				(size 1 1)
+			)
+			(justify left)
+		)
+		(property "Intersheetrefs" "${INTERSHEET_REFS}"
+			(at 205.74 54.61 0)
+			(hide yes)
+			(show_name no)
+			(do_not_autoplace no)
+			(effects
+				(font
+					(size 1.27 1.27)
+				)
+			)
+		)
+	)
+	(wire
+		(pts
+			(xy 250.19 129.54) (xy 274.32 129.54)
+		)
+		(stroke
+			(width 0)
+			(type default)
+		)
+	)
+	(global_label "LDAC_N"
+		(shape passive)
+		(at 255.27 129.54 0)
+		(effects
+			(font
+				(size 1 1)
+			)
+			(justify left)
+		)
+		(property "Intersheetrefs" "${INTERSHEET_REFS}"
+			(at 255.27 129.54 0)
+			(hide yes)
+			(show_name no)
+			(do_not_autoplace no)
+			(effects
+				(font
+					(size 1.27 1.27)
+				)
+			)
+		)
+	)
+	(global_label "STAR"
+		(shape passive)
+		(at 274.32 129.54 0)
+		(effects
+			(font
+				(size 1 1)
+			)
+			(justify left)
+		)
+		(property "Intersheetrefs" "${INTERSHEET_REFS}"
+			(at 274.32 129.54 0)
+			(hide yes)
+			(show_name no)
+			(do_not_autoplace no)
+			(effects
+				(font
+					(size 1.27 1.27)
+				)
+			)
+		)
+	)
+	(wire
+		(pts
+			(xy 250.19 137.16) (xy 274.32 137.16)
+		)
+		(stroke
+			(width 0)
+			(type default)
+		)
+	)
+	(global_label "COIL_COM"
+		(shape passive)
+		(at 255.27 137.16 0)
+		(effects
+			(font
+				(size 1 1)
+			)
+			(justify left)
+		)
+		(property "Intersheetrefs" "${INTERSHEET_REFS}"
+			(at 255.27 137.16 0)
+			(hide yes)
+			(show_name no)
+			(do_not_autoplace no)
+			(effects
+				(font
+					(size 1.27 1.27)
+				)
+			)
+		)
+	)
+	(global_label "+5V_An"
+		(shape passive)
+		(at 274.32 137.16 0)
+		(effects
+			(font
+				(size 1 1)
+			)
+			(justify left)
+		)
+		(property "Intersheetrefs" "${INTERSHEET_REFS}"
+			(at 274.32 137.16 0)
+			(hide yes)
+			(show_name no)
+			(do_not_autoplace no)
+			(effects
+				(font
+					(size 1.27 1.27)
+				)
+			)
+		)
+	)
 )
